File: Face2/Face2.kicad_pcb (KiCad board)
At the start: 2 copper layers, 99.1 x 99.1 mm, 6 parts, among them J1 Conn_02x04_Counter_Clockwise, J2 Conn_02x04_Counter_Clockwise

Commit message: Changed to multiple AS1105 for LED drivers
Parts:
- J1: value Conn_02x04_Counter_Clockwise -> Conn_02x04_Odd_Even
- J2: value Conn_02x04_Counter_Clockwise -> Conn_01x04_Male; footprint Connector_IDC:IDC-Header_2x04_P2.54mm_Vertical -> Connector:FanPinHeader_1x04_P2.54mm_Vertical
- moved J1 5.86 mm to (124.0, 79.2)
- moved J2 4.85 mm to (175.8, 74.7), turned to 270 degrees
Connections:
- D1 pad 1: DIG4 -> DIG0
- D2 pad 1: DIG4 -> DIG0
- D3 pad 1: DIG4 -> DIG0
- D4 pad 1: DIG4 -> DIG0
- J1 pad 2: SEGB -> SEGDP
- J1 pad 3: SEGC -> SEGB
- J1 pad 4: SEGD -> SEGG
- J1 pad 5: SEGE -> SEGC
- J1 pad 7: SEGG -> SEGD
- J1 pad 8: SEGDP -> SEGE
Routing:
- net DIG4: track 44.1 -> 0.00 mm
- net DIG0: track 0.00 -> 44.1 mm
